Commit message: some changes

File: irobot_create_common/irobot_create_description/urdf/create3.urdf.xacro (robot description, xacro)
@@ -84,5 +84,5 @@
     <parent link="base_link"/>
     <child link="sensor_box"/>
-    <origin xyz="-0.02 0 0.115" rpy="0 0 0"/>
+    <origin xyz="0.0 0 0.110" rpy="0 0 0"/>
   </joint>
   <link name="sensor_box">
@@ -96,8 +96,8 @@
       <origin xyz="0 0 0" rpy="0 0 0"/>
       <geometry>
-        <box size="0.1 0.1 0.04"/>
+        <box size="0.1 0.1 0.05"/>
       </geometry>
     </collision>
-    <xacro:inertial_cuboid_with_pose mass="0.2" x="0.1" y="0.1" z="0.04">
+    <xacro:inertial_cuboid_with_pose mass="0.2" x="0.1" y="0.1" z="0.05">
       <origin xyz="0 0 0" />
     </xacro:inertial_cuboid_with_pose>
@@ -105,5 +105,6 @@
   <!-- Camera -->
   <xacro:sensor_d435i parent="base_link" use_nominal_extrinsics="true">
-    <origin xyz="0.02 0 0.115" rpy="0 0 0" />
+    <!-- <origin xyz="0.02 0 0.115" rpy="0 0 0" /> -->
+    <origin xyz="0.059 0 0.110" rpy="0 0 0"/>
   </xacro:sensor_d435i>
   <!-- Bumper -->

File: irobot_create_common/irobot_create_description/urdf/sensor_box.urdf.xacro (robot description, xacro)
@@ -5,4 +5,18 @@
       <color rgba="0.2 0.2 1 1"/>
     </material>
+    <link name="sensor_box">
+        <visual>
+            <geometry>
+            <box size="0.1 0.1 0.05"/>
+            </geometry>
+            <material name="blue"/>
+        </visual>
+    </link>
+    <joint name="box_joint" type="fixed">
+        <parent link="base_link"/>
+        <child link="sensor_box"/>
+        <origin xyz="0 0 0.0.110" rpy="0 0 0"/>
+    </joint>
+<!--
     <joint name="sensor_box" type="fixed">
         <parent link="base_link"/>
@@ -61,4 +75,4 @@
             </plugin>
         </sensor>
-    </gazebo>
+    </gazebo> -->
 </robot>

File: irobot_create_common/irobot_create_description/urdf/sensors/camera.xacro (robot description, xacro)
@@ -3,4 +3,5 @@
     <joint name="camera_joint" type="fixed">
         <origin xyz="0 0 0" rpy="0 0 0"/>
+        <!-- <origin xyz="0.059 0 0.040" rpy="0 0 -3.1416"/> -->
         <parent link="base_link"/>
         <child link="camera_link" />

File: irobot_create_common/irobot_create_description/urdf/sensors/lidar.urdf.xacro (robot description, xacro)
@@ -8,5 +8,6 @@
         <parent link="base_link"/>
         <child link="laser_frame"/>
-        <origin xyz="-0.02 0 0.16" rpy="0 0 0"/>
+        <!-- <origin xyz="-0.02 0 0.16" rpy="0 0 0"/> -->
+        <origin xyz="-0.009 0 0.15" rpy="0 0 3.1416"/>
     </joint>
     <link name="laser_frame">
